File: kicad-template_1590BB.kicad_pcb (KiCad board)
At the start: 2 copper layers, 0 parts

Commit message: updated 1590BB layout to landscape
Parts:
- added J1: Barrel_Jack_Switch, bca-footprints:DC_Jack_DC005, F.Cu at (0.00, -43.5)
- added J2: AudioJack_TRS, bca-footprints:Rean_NYS215, F.Cu at (-36.0, -30.0)
- added J3: AudioJack_TRS, bca-footprints:Rean_NYS215, F.Cu at (36.0, -30.0)
Other:
- board outline added: 110 x 84.3 mm
- net class Default: trace_width 0.1 -> 0.25
- rule trace_min: 0.1 -> 0.2
